Commit message: 3link 2joint

File: body.urdf (robot description, URDF)
Before this commit: robot robot, 2 links, 1 joints
Links:
- added link Link2, mass 1; collision box size=1 1 1; visual box size=1 1 1
Joints:
- added joint Link1_Link2: type revolute, parent Link1, child Link2, origin xyz=1 0 0 rpy=0 0 0, axis 0 1 0, limit lower=-3.14159 upper=3.14159 effort=0.0 velocity=0.0

Commit message: sensors

File: body.urdf (robot description, URDF)
Before this commit: robot robot, 3 links, 2 joints
Links:
- removed link Link0
- removed link Link1
- removed link Link2
- added link Backleg, mass 1; collision box size=1 1 1; visual box size=1 1 1
- added link Frontleg, mass 1; collision box size=1 1 1; visual box size=1 1 1
- added link Torso, mass 1; collision box size=1 1 1; visual box size=1 1 1
Joints:
- removed joint Link0_Link1
- removed joint Link1_Link2
- added joint Torso_Backleg: type revolute, parent Torso, child Backleg, origin xyz=-0.5 0 1 rpy=0 0 0, axis 0 1 0, limit lower=-3.14159 upper=3.14159 effort=0.0 velocity=0.0
- added joint Torso_Frontleg: type revolute, parent Torso, child Frontleg, origin xyz=0.5 0 1 rpy=0 0 0, axis 0 1 0, limit lower=-3.14159 upper=3.14159 effort=0.0 velocity=0.0
